Commit message: All random changes so far for troubleshooting

File: src/marsarm_moveit/urdf/marsarm.urdf (robot description, URDF)
Before this commit: robot Mars_Arm, 10 links, 9 joints
Links:
- link base: geometry visual cylinder length=0.3 radius=0.06
- link elbow: geometry visual cylinder length=0.15 radius=0.04
- link forearm: geometry visual cylinder length=0.3 radius=0.06
- link hand: geometry visual cylinder length=0.1 radius=0.04
- link main_arm: geometry visual cylinder length=0.3 radius=0.06
- link shoulder: geometry visual cylinder length=0.15 radius=0.04
- link wrist: geometry visual cylinder length=0.15 radius=0.04
